File: pcb/wideband_v2/wideband_v2.kicad_sch (KiCad schematic)
At the start: 57 parts, among them J1 DISPLAY, J2 GPIO, J3 LSU, J4 Tag connect, J5 USB, SW1 SW_Push, U1 MCP4725xxx-xCH, U2 L7805, U3 MCP4725xxx-xCH, U4 RP2040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

Commit message: Updating BOM SKUs
Parts:
- D4: value BLUE -> RED
- R1, R2, R3: LCSC C11702 -> (none)
Changed lines of the file:
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@@
-      (effects (font (size 1.27 1.27)) hide)
-    )
-    (property "LCSC" "C11702" (id 4) (at 38.735 130.81 90)
       (effects (font (size 1.27 1.27)) hide)
     )
@@
       (effects (font (size 1.27 1.27)) hide)
     )
-    (property "LCSC" "C11702" (id 4) (at 38.735 121.92 90)
-      (effects (font (size 1.27 1.27)) hide)
-    )
     (pin "1")
     (pin "2")
@@
     )
     (property "Datasheet" "~" (id 3) (at 38.735 113.03 0)
-      (effects (font (size 1.27 1.27)) hide)
-    )
-    (property "LCSC" "C11702" (id 4) (at 38.735 113.03 90)
       (effects (font (size 1.27 1.27)) hide)
     )
@@
       (effects (font (size 1.27 1.27)) (justify right))
     )
-    (property "Value" "BLUE" (id 1) (at 28.575 133.35 0)
+    (property "Value" "RED" (id 1) (at 28.575 133.35 0)
       (effects (font (size 1.27 1.27)) (justify right))
     )
@@
     )
     (path "/f5339ee5-a7dd-44be-a314-2d5cfa5bc702"
-      (reference "D4") (unit 1) (value "BLUE") (footprint "LED_SMD:LED_0603_1608Metric")
+      (reference "D4") (unit 1) (value "RED") (footprint "LED_SMD:LED_0603_1608Metric")
     )
     (path "/2371badf-0abe-4616-95ad-e750dddfceb3"

Commit message: MCP4725 => DAC5571
Parts:
- removed U1, U3: MCP4725xxx-xCH, Package_TO_SOT_SMD:SOT-23-6, symbol Analog_DAC:MCP4725xxx-xCH
- added U1, U3: DAC5571IDBVR, Package_TO_SOT_SMD:SOT-23-6, symbol Analog_DAC:DAC081C081CIMK
Connections:
- net +5V: now also U1.3 (GND), U3.3 (GND), U3.6 (ADR0)
- net D_SCL_5: now also U1.5 (SCL), U3.5 (SCL)
- net D_SDA_5: now also U1.4 (SDA), U3.4 (SDA)
- net GND: now also U1.2 (VA), U1.6 (ADR0), U3.2 (VA)
- net V0: now also U1.1 (VOUT)
- net V1: now also U3.1 (VOUT)

Commit message: add CAN controller
Parts:
- added C36, C37: 30pF, Capacitor_SMD:C_0603_1608Metric, symbol Device:C_Small
- added C38: 4.7nF, Capacitor_SMD:C_0805_2012Metric, symbol Device:C_Small
- added R35: 10k, Resistor_SMD:R_0603_1608Metric, symbol Device:R
- added R36, R37: R_Small, Resistor_SMD:R_1206_3216Metric, symbol Device:R_Small
- added U11: MCP2515-xSO, Package_SO:SOIC-18W_7.5x11.6mm_P1.27mm, symbol Interface_CAN_LIN:MCP2515-xSO
- added U12: TJA1042T3118, Package_SO:HTSOP-8-1EP_3.9x4.9mm_P1.27mm_EP2.4x3.2mm, symbol OpenEFI-STM32-rev3:TJA1042T3118
- added Y2: 12MHz, Crystal:Crystal_SMD_3225-4Pin_3.2x2.5mm, symbol Device:Crystal_GND24
Connections:
- net +3V3: now also R35.2, U11.18 (VDD), U12.5 (VIO)
- net +5V: now also U12.3 (VCC)
- net GND: now also C36.1, C37.1, C38.2, U11.9 (VSS), U12.2 (GND), U12.8 (STB), Y2.2, Y2.4; no longer J3.7 (Pin_7)
- net GPIO0: now also U11.13 (SCK)
- net GPIO1: now also U11.14 (SI)
- net GPIO3: now also U11.15 (SO)
- net V0: now also J3.5 (Pin_5); no longer J3.11 (Pin_11)
- net V1: now also J3.7 (Pin_7); no longer J3.12 (Pin_12)
- net GPIO8: now reaches U4.11 (GPIO8)
- net GPIO8: now also U11.16 (~{CS})
- new net: C38.1, R36.1, R37.1
- new net: R35.1, U11.17 (~{RESET})
- new net: U11.2 (RXCAN), U12.1 (TXD)
- new net: U11.1 (TXCAN), U12.4 (RXD)
- new net CAN+: J3.11 (Pin_11), R36.2, U12.7 (CANH)
- new net CAN-: J3.12 (Pin_12), R37.2, U12.6 (CANL)
- new net CAN_CLOCK_A: C36.2, U11.8 (OSC1), Y2.3
- new net CAN_CLOCK_B: C37.2, U11.7 (OSC2), Y2.1
- no-connect marks 7 -> 5
Other:
- moved on the sheet: U6

Commit message: trace external i/o
Parts:
- removed C10: 100nF, Capacitor_SMD:C_0603_1608Metric, symbol Device:C_Small
Changed lines of the file:
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@@
     (pin "1")
-  )
-  (symbol (lib_id "Device:C_Small") (at 203.2 22.86 0) (unit 1)
-    (in_bom yes) (on_board yes)
-    (property "Reference" "C10" (id 0) (at 203.2 20.32 0)
-      (effects (font (size 1.27 1.27)) (justify left))
-    )
-    (property "Value" "100nF" (id 1) (at 204.47 26.67 0)
-      (effects (font (size 1.27 1.27)) (justify left))
-    )
-    (property "Footprint" "Capacitor_SMD:C_0603_1608Metric" (id 2) (at 203.2 22.86 0)
-      (effects (font (size 1.27 1.27)) hide)
-    )
-    (property "Datasheet" "~" (id 3) (at 203.2 22.86 0)
-      (effects (font (size 1.27 1.27)) hide)
-    )
-    (pin "1")
-    (pin "2")
   )
   (symbol (lib_id "power:+1V1") (at 176.53 29.21 0) (unit 1)
@@
       (reference "C9") (unit 1) (value "2.2uF") (footprint "Capacitor_SMD:C_0603_1608Metric")
     )
-    (path "/1557a4a3-ef96-4959-8260-1ee82b8b664b"
-      (reference "C10") (unit 1) (value "100nF") (footprint "Capacitor_SMD:C_0603_1608Metric")
-    )
     (path "/3a596820-bd87-4d20-8890-43c438853180"

Commit message: Routing
Parts:
- R36, R37: value R_Small -> 30R
Connections:
- net GPIO2: now also U11.15 (SO)
- net GPIO3: no longer U11.15 (SO)
- no-connect marks 5 -> 12
Other:
- moved on the sheet: C36, C37, C38, J2, R35, R36, R37, U11, U12, Y2
