File: pcb/wideband_v3/Wideband_v3/Wideband_v3.kicad_pcb (KiCad board)
At the start: 2 copper layers, 85 x 77.9 mm, 76 parts, among them J1 Conn_01x10, J2 USB_C_Receptacle_USB2.0, J3 Tag connect, J4 FT_CAN, J5 Conn_01x12, Q1 SS8050, Q2 IRLZ44N, Q3 IRLZ44N, SW1 Key0, SW3 Key1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

Commit message: update pcb layout
Parts:
- added D7: 1N4148W, Diode_SMD:D_SOD-123, F.Cu at (177.8, 93.3)
- added H1: MountingHole, MountingHole:MountingHole_3.2mm_M3_Pad_Via, F.Cu at (151.1, 71.8)
- added H2: MountingHole, MountingHole:MountingHole_3.2mm_M3_Pad_Via, F.Cu at (83.8, 71.1)
- added H3: MountingHole, MountingHole:MountingHole_3.2mm_M3_Pad_Via, F.Cu at (82.5, 109.9)
- added H4: MountingHole, MountingHole:MountingHole_3.2mm_M3_Pad_Via, F.Cu at (151.8, 110.5)
- added R17: 33k, Resistor_SMD:R_0603_1608Metric, F.Cu at (200.9, 113.7)
- added R18: 15k, Resistor_SMD:R_0603_1608Metric, F.Cu at (200.9, 116.2)
- added U10: LMV358, Package_SO:SOIC-8_3.9x4.9mm_P1.27mm, F.Cu at (189.9, 102.2)
- J4, J5: moved to B.Cu
- SW1: footprint Button_Switch_THT:SW_SPST_Omron_B3F-315x_Angled -> Button_Switch_SMD:SW_Push_1P1T_XKB_TS-1187A
- moved U9 87.3 mm to (189.2, 113.0)
- moved C3 83.1 mm to (224.2, 113.8)
- moved C4 83.1 mm to (236.5, 114.0)
- moved C5 83.1 mm to (236.5, 117.0)
- moved C6 83.1 mm to (215.2, 123.8)
- moved D1 83.1 mm to (236.5, 122.8)
- moved D2 83.1 mm to (236.5, 125.3)
- moved D3 83.1 mm to (230.2, 114.8)
- moved D4 83.1 mm to (230.2, 119.3)
- moved Q3 83.1 mm to (216.9, 115.7)
- moved R10 83.1 mm to (224.2, 121.3)
- moved R12 83.1 mm to (224.2, 123.8)
- moved R13 83.1 mm to (224.2, 126.3)
- moved R14 83.1 mm to (224.2, 128.8)
- moved R7 83.1 mm to (234.0, 129.6)
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Connections:
- J5 pad 4: +12VA -> /NARROW
- U1 pad 12: unconnected-(U1-GPIO9-Pad12) -> /CAN_TX
- U1 pad 13: unconnected-(U1-GPIO10-Pad13) -> /CAN_RX
- U1 pad 34: unconnected-(U1-GPIO22-Pad34) -> /DAC_SCK
- U1 pad 35: /MCU/BT_CS -> /DAC_CS
- U1 pad 36: unconnected-(U1-GPIO24-Pad36) -> /DAC_SO
- U1 pad 37: unconnected-(U1-GPIO25-Pad37) -> /DAC_SI
- U1 pad 39: unconnected-(U1-GPIO27_ADC1-Pad39) -> /m_narrow
- U1 pad 40: unconnected-(U1-GPIO28_ADC2-Pad40) -> /MCU/WBO_RX
- U1 pad 41: unconnected-(U1-GPIO29_ADC3-Pad41) -> /MCU/WBO_TX
Other:
- board size 85 x 77.9 mm -> 80 x 50 mm

Commit message: init 7seg pcb
Parts:
- removed C3: 47nF, Capacitor_SMD:C_0603_1608Metric
- removed C4: 100nF, Capacitor_SMD:C_0805_2012Metric
- removed C5: 10nF, Capacitor_SMD:C_0805_2012Metric
- removed C6: 330uF ±20% 6.3V, Capacitor_SMD:CP_Elec_6.3x7.7
- removed D3: SMAJ58CA, Diode_SMD:D_SMA
- removed D4: B540C-13-F, Diode_SMD:D_SMA
- removed L1: 10uH, Inductor_SMD:L_7.3x7.3_H4.5
- removed Q1: SS8050, Package_TO_SOT_SMD:SOT-23
- removed Q2, Q3: IRLZ44N, Package_TO_SOT_SMD:TO-252-2
- removed R10, R8: 10R 1/10W, Resistor_SMD:R_0603_1608Metric
- removed R11: 0.01R, Resistor_SMD:R_1210_3225Metric
- removed R12: 57.6K 1/10W, Resistor_SMD:R_0603_1608Metric
- removed R13: 4.99K 1/10W, Resistor_SMD:R_0603_1608Metric
- removed R14: 10k, Resistor_SMD:R_0603_1608Metric
- removed R15: 3.24k, Resistor_SMD:R_0603_1608Metric
- removed R7: 10k, Resistor_SMD:R_0805_2012Metric
- removed R9: 1M 1/10W, Resistor_SMD:R_0603_1608Metric
- removed TP1: SWCLK, TestPoint:TestPoint_Pad_1.0x1.0mm
- removed TP2: SWD, TestPoint:TestPoint_Pad_1.0x1.0mm
- removed U5: LT4363IMS, Package_SO:MSOP-12_3x4mm_P0.65mm
- removed U6: TPS5430DDA, Package_SO:TI_SO-PowerPAD-8_ThermalVias
- added C28: 1u, Capacitor_SMD:C_0603_1608Metric, F.Cu at (111.8, 108.4)
- added C29: 1u, Capacitor_SMD:C_0603_1608Metric, F.Cu at (124.8, 110.2)
- added C30: 22u, Capacitor_SMD:C_0805_2012Metric, F.Cu at (122.9, 110.1)
- added D10: D_TVS, Diode_SMD:D_SMC, F.Cu at (102.7, 106.5)
- added D11: BZV55B20, Diode_SMD:D_MiniMELF, F.Cu at (110.8, 110.4)
- added G***: LOGO, LOGO, F.Cu at (93.2, 104.9)
- added G***: LOGO, LOGO, F.Cu at (143.8, 108.9)
- added G***: LOGO, LOGO, B.Cu at (103.3, 103.7)
- added G***: LOGO, LOGO, B.Cu at (140.5, 104.9)
- added G***: LOGO, LOGO, B.Cu at (112.0, 84.3)
- added Q6: MCQ9435-TP, Package_SO:SOIC-8_3.9x4.9mm_P1.27mm, F.Cu at (110.1, 104.3)
- added R19: 10k, Resistor_SMD:R_0603_1608Metric, F.Cu at (140.9, 99.5)
- added R20: 10k, Resistor_SMD:R_0603_1608Metric, F.Cu at (112.8, 100.7)
- added U11: LM78M05_TO252, Package_TO_SOT_SMD:TO-252-2, F.Cu at (118.1, 105.5)
- D1, D2: value 1N4148 -> B120-E3; footprint Diode_SMD:D_SOD-523 -> Diode_SMD:D_SMA
- D5, D6, D7: footprint Diode_SMD:D_SOD-123 -> Diode_SMD:D_SOD-323F
- JP1, JP2, JP3, JP5, SW1, TP3: moved to B.Cu
- moved D2 114.9 mm to (123.5, 104.3), turned to -90 degrees
- moved R18 114.0 mm to (88.0, 99.9), turned to -90 degrees
- moved R17 109.2 mm to (93.4, 94.1), turned to -90 degrees
- moved C7 104.3 mm to (92.7, 99.9), turned to 180 degrees
- moved U9 103.7 mm to (89.7, 83.8), turned to -90 degrees
- moved D1 101.3 mm to (136.4, 107.6), turned to -90 degrees
- moved U10 100.4 mm to (89.8, 94.4), turned to -90 degrees
- moved U8 92.7 mm to (130.7, 106.8), turned to 90 degrees
- moved U2 88.6 mm to (131.4, 96.4), turned to 45 degrees
- moved D7 88.1 mm to (89.9, 100.0), turned to 90 degrees
- moved JP5 83.9 mm to (103.2, 80.3)
- moved R6 83.7 mm to (126.6, 95.7), turned to -135 degrees
- moved JP4 82.7 mm to (125.9, 99.4), turned to 135 degrees
- moved C16 81.5 mm to (145.0, 84.2), turned to 135 degrees
- moved U1 81.1 mm to (139.4, 86.1), turned to 135 degrees
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Connections:
- D1 pad 1: Net-(D1-K) -> +5V
- D1 pad 2: +12VA -> VBUS
- D2 pad 1: Net-(D2-K) -> +5V
- D2 pad 2: GND -> Net-(D2-A)
- J1 pad 11: VBUS -> +5V
- J1 pad 7: /MCU/GPIO10 -> /MCU/GPIO16
- J5 pad 1: +12V -> /HEATER-
- J5 pad 2: /HEATER- -> +12VA
- J5 pad 3: +12VA -> +12V
- U1 pad 24: Net-(U1-SWCLK) -> /MCU/SYS_SWCLK
- U1 pad 25: Net-(U1-SWD) -> /MCU/SYS_SWDIO
- U1 pad 26: +3V3 -> /MCU/NRST
Routing:
- net +5V: track 0.00 -> 175.3 mm, vias 0 -> 8
- net +3V3: track 0.00 -> 147.1 mm, vias 0 -> 15
- net /MCU/GPIO16: track 0.00 -> 87.7 mm, vias 0 -> 1
- net /MCU/GPIO14: track 0.00 -> 82.6 mm, vias 0 -> 1
- net /MCU/GPIO8: track 0.00 -> 81.8 mm, vias 0 -> 2
- net /MCU/GPIO12: track 0.00 -> 81.6 mm, vias 0 -> 1
- net /MCU/GPIO11: track 0.00 -> 80.0 mm, vias 0 -> 1
- net /MCU/GPIO7: track 0.00 -> 75.1 mm, vias 0 -> 1
- net +12V: track 0.00 -> 69.6 mm
- net /MCU/GPIO26: track 0.00 -> 64.2 mm, vias 0 -> 1
- net /m_narrow: track 0.00 -> 62.2 mm, vias 0 -> 2
- net /MCU/GPIO21: track 0.00 -> 61.1 mm, vias 0 -> 1
- net /m_TEMP_OUT: track 0.00 -> 45.6 mm, vias 0 -> 2
- net /m_LAMBDA_OUT: track 0.00 -> 42.8 mm, vias 0 -> 2
- net /NARROW: track 0.00 -> 38.4 mm, vias 0 -> 1
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- added copper zone on In1.Cu, net +3V3
- added copper zone on In2.Cu, net +3V3
- added copper zone on B.Cu, net GND
- added copper zone on F.Cu, net GND
- added copper zone on In1.Cu, net GND
- added copper zone on In2.Cu, net GND
Other:
- copper layers 2 -> 4
- board text added: "Churrosoft"
- board text added: "Diseñado en Argentina"
- board text added: "OpenEFI Wideband v3.x"
- board text added: "®"

Commit message: Cosas
Parts:
- moved SW1 1.33 mm to (126.8, 83.5)
- moved C19 0.59 mm to (135.7, 90.8)
- moved C11 0.48 mm to (134.6, 91.9)
- moved C23 0.35 mm to (135.4, 80.8)
- moved C16 0.34 mm to (145.3, 84.3)
- moved R5 0.33 mm to (140.1, 93.6)
Connections:
- J1 pad 10: +3V3 -> +12VA
- J1 pad 2: /MCU/GPIO26 -> /MCU/GPIO21
- J1 pad 3: /MCU/GPIO21 -> /MCU/GPIO20
- J1 pad 4: /MCU/GPIO14 -> /MCU/GPIO19
- J1 pad 5: /MCU/GPIO12 -> /MCU/GPIO18
- J1 pad 6: /MCU/GPIO11 -> /MCU/GPIO17
- J1 pad 8: /MCU/GPIO8 -> /MCU/GPIO15
- J1 pad 9: /MCU/GPIO7 -> /MCU/GPIO14
- JP4 pad 2: Net-(JP4-B) -> /MCU/FORCE_BOOTLOADER
- R6 pad 2: Net-(JP4-B) -> /MCU/FORCE_BOOTLOADER
- SW1 pad 2: Net-(U1-GPIO15) -> /MCU/FORCE_BOOTLOADER
- SW3 pad 2: Net-(U1-GPIO18) -> /MCU/BTN_YES
- U1 pad 18: Net-(U1-GPIO15) -> /MCU/GPIO15
- U1 pad 28: unconnected-(U1-GPIO17-Pad28) -> /MCU/GPIO17
- U1 pad 29: Net-(U1-GPIO18) -> /MCU/GPIO18
- U1 pad 5: unconnected-(U1-GPIO3-Pad5) -> /MCU/BTN_YES
Routing:
- net /MCU/GPIO8: track 81.8 -> 0.00 mm, vias 2 -> 0
- net /MCU/GPIO12: track 81.6 -> 0.00 mm, vias 1 -> 0
- net /MCU/GPIO11: track 80.0 -> 0.00 mm, vias 1 -> 0
- net /MCU/GPIO7: track 75.1 -> 0.00 mm, vias 1 -> 0
- net /MCU/GPIO15: track 0.00 -> 72.6 mm, vias 0 -> 1
- net /MCU/GPIO18: track 0.00 -> 71.7 mm, vias 0 -> 1
- net /MCU/GPIO20: track 0.00 -> 69.8 mm, vias 0 -> 1
- net /MCU/GPIO19: track 0.00 -> 69.6 mm, vias 0 -> 1
- net /MCU/GPIO17: track 0.00 -> 69.2 mm, vias 0 -> 1
- net /MCU/GPIO26: track 64.2 -> 0.00 mm, vias 1 -> 0
- net GND: track 29.5 -> 93.4 mm, vias 7 -> 17
- net +12VA: track 37.5 -> 67.1 mm
- net Net-(U1-GPIO15): track 24.0 -> 0.00 mm, vias 1 -> 0
- net +3V3: track 147.1 -> 169.6 mm
- net +5V: track 175.3 -> 154.8 mm, vias 8 -> 5
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- removed copper zone on In1.Cu, net +3V3
- removed copper zone on In2.Cu, net +3V3
- removed copper zone on In1.Cu, net GND
- removed copper zone on In2.Cu, net GND
Other:
- copper layers 4 -> 2
