File: pcb/wideband_v3/Wideband_v3/Wideband_v3.kicad_sch (KiCad schematic)
At the start: 18 parts, among them J4 FT_CAN, J5 Conn_01x12, U10 LMV358, U4 TJA1051T-3, U7 MCP42010, U9 LMV358

Commit message: update pcb layout
Parts:
- U10: footprint (none) -> Package_SO:SOIC-8_3.9x4.9mm_P1.27mm
Changed lines of the file:
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@@
-    (stroke (width 0) (type default))
-  )
-  (wire (pts (xy 137.16 144.78) (xy 137.16 146.05))
     (stroke (width 0) (type default))
   )
@@
   (text "los mini-fit HCS en teoria\nbancan hasta 13A asi que este \njoputa tendria que aguantar 3A \nsin derretirse (opcional)" (exclude_from_sim no)
     (at 229.362 128.016 0)
-    (effects (font (face "Source Code Pro") (size 0.8 0.8)))
+    (effects (font (face "Vazirmatn") (size 0.9 0.9)))
   )
   (text "estos pines los puse medio al tuntun,\nsi podes revisa si alguno no esta para el culo" (exclude_from_sim no)
@@
       (effects (font (size 1.27 1.27)) (justify left))
     )
-    (property "Footprint" "" (at 166.37 152.4 0)
+    (property "Footprint" "Package_SO:SOIC-8_3.9x4.9mm_P1.27mm" (at 166.37 152.4 0)
       (effects (font (size 1.27 1.27)) hide)
     )
@@
       (effects (font (size 1.27 1.27)))
     )
-    (property "Footprint" "" (at 234.95 86.36 0)
+    (property "Footprint" "Package_SO:SOIC-8_3.9x4.9mm_P1.27mm" (at 234.95 86.36 0)
       (effects (font (size 1.27 1.27)) hide)
     )
@@
       (effects (font (size 1.27 1.27)))
     )
-    (property "Footprint" "" (at 199.39 87.63 0)
-      (effects (font (size 1.27 1.27)) hide)
-    )
+    (property "Footprint" "Package_SO:SOIC-8_3.9x4.9mm_P1.27mm" (at 199.39 87.63 0)
+      (effects (font (size 1.27 1.27)) hide)
+    )

Commit message: init 7seg pcb
Parts:
- D5, D6, D7: footprint Diode_SMD:D_SOD-123 -> Diode_SMD:D_SOD-323F
- J4: LCSC (none) -> C586650
Connections:
- net +12V: now also J5.3 (Pin_3); no longer J5.1 (Pin_1)
- net +12VA: now also J5.2 (Pin_2); no longer J5.3 (Pin_3)
- net HEATER-: now also J5.1 (Pin_1); no longer J5.2 (Pin_2)
