File: pcb/wideband_v3/Wideband_v3/mcu.kicad_sch (KiCad schematic)
At the start: 38 parts, among them J1 Conn_01x10, J2 USB_C_Receptacle_USB2.0, J3 Tag connect, SW1 Key0, SW3 Key1, U1 RP2040, U2 W25Q128JVS, U8 AMS1117-3.3, Y1 12MHz

Commit message: update pcb layout
Parts:
- added H1, H2, H3, H4: MountingHole, MountingHole:MountingHole_3.2mm_M3_Pad_Via, symbol Mechanical:MountingHole
- SW1: footprint Button_Switch_THT:SW_SPST_Omron_B3F-315x_Angled -> Button_Switch_SMD:SW_Push_1P1T_XKB_TS-1187A
Changed lines of the file:
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@@
+    )
+  )
+  (symbol (lib_id "Mechanical:MountingHole") (at 69.85 177.8 0) (unit 1)
+    (exclude_from_sim no) (in_bom yes) (on_board yes) (dnp no) (fields_autoplaced)
+    (property "Reference" "H4" (at 72.39 176.5299 0)
+      (effects (font (size 1.27 1.27)) (justify left))
+    )
+    (property "Value" "MountingHole" (at 72.39 179.0699 0)
+      (effects (font (size 1.27 1.27)) (justify left))
+    )
+    (property "Footprint" "MountingHole:MountingHole_3.2mm_M3_Pad_Via" (at 69.85 177.8 0)
+      (effects (font (size 1.27 1.27)) hide)
+    )
+    (property "Datasheet" "~" (at 69.85 177.8 0)
+      (effects (font (size 1.27 1.27)) hide)
+    )
+    (property "Description" "Mounting Hole without connection" (at 69.85 177.8 0)
+      (effects (font (size 1.27 1.27)) hide)
+    )
+    (instances
+      (project "Wideband_v3"
+        (path "/08893845-3ad0-4661-81a4-b965d2c3e6dc/3737bf71-68b2-46c2-b6f0-6262322b912b"
+          (reference "H4") (unit 1)
+        )
+      )
     )
   )
@@
     )
   )
+  (symbol (lib_id "Mechanical:MountingHole") (at 60.9978 167.0456 0) (unit 1)
+    (exclude_from_sim no) (in_bom yes) (on_board yes) (dnp no) (fields_autoplaced)
+    (property "Reference" "H2" (at 63.5378 165.7755 0)
+      (effects (font (size 1.27 1.27)) (justify left))
+    )
+    (property "Value" "MountingHole" (at 63.5378 168.3155 0)
+      (effects (font (size 1.27 1.27)) (justify left))
+    )
+    (property "Footprint" "MountingHole:MountingHole_3.2mm_M3_Pad_Via" (at 60.9978 167.0456 0)
+      (effects (font (size 1.27 1.27)) hide)
+    )
+    (property "Datasheet" "~" (at 60.9978 167.0456 0)
+      (effects (font (size 1.27 1.27)) hide)
+    )
+    (property "Description" "Mounting Hole without connection" (at 60.9978 167.0456 0)
+      (effects (font (size 1.27 1.27)) hide)
+    )
+    (instances
+      (project "Wideband_v3"
+        (path "/08893845-3ad0-4661-81a4-b965d2c3e6dc/3737bf71-68b2-46c2-b6f0-6262322b912b"
+          (reference "H2") (unit 1)
+        )
+      )
+    )
+  )
   (symbol (lib_id "power:GND") (at 200.66 106.68 0) (unit 1)
     (exclude_from_sim no) (in_bom yes) (on_board yes) (dnp no) (fields_autoplaced)
@@
     )
   )
+  (symbol (lib_id "Mechanical:MountingHole") (at 62.23 161.29 0) (unit 1)
+    (exclude_from_sim no) (in_bom yes) (on_board yes) (dnp no) (fields_autoplaced)
+    (property "Reference" "H1" (at 64.77 160.0199 0)
+      (effects (font (size 1.27 1.27)) (justify left))
+    )
+    (property "Value" "MountingHole" (at 64.77 162.5599 0)
+      (effects (font (size 1.27 1.27)) (justify left))
+    )
+    (property "Footprint" "MountingHole:MountingHole_3.2mm_M3_Pad_Via" (at 62.23 161.29 0)
+      (effects (font (size 1.27 1.27)) hide)
+    )
+    (property "Datasheet" "~" (at 62.23 161.29 0)
+      (effects (font (size 1.27 1.27)) hide)
+    )
+    (property "Description" "Mounting Hole without connection" (at 62.23 161.29 0)
+      (effects (font (size 1.27 1.27)) hide)
+    )
+    (instances
+      (project "Wideband_v3"
+        (path "/08893845-3ad0-4661-81a4-b965d2c3e6dc/3737bf71-68b2-46c2-b6f0-6262322b912b"
+          (reference "H1") (unit 1)
+        )
+      )
+    )
+  )
   (symbol (lib_id "power:GND") (at 151.13 148.59 0) (unit 1)
     (exclude_from_sim no) (in_bom yes) (on_board yes) (dnp no) (fields_autoplaced)
@@
     )
   )
+  (symbol (lib_id "Mechanical:MountingHole") (at 60.96 172.72 0) (unit 1)
+    (exclude_from_sim no) (in_bom yes) (on_board yes) (dnp no) (fields_autoplaced)
+    (property "Reference" "H3" (at 63.5 171.4499 0)
+      (effects (font (size 1.27 1.27)) (justify left))
+    )
+    (property "Value" "MountingHole" (at 63.5 173.9899 0)
+      (effects (font (size 1.27 1.27)) (justify left))
+    )
+    (property "Footprint" "MountingHole:MountingHole_3.2mm_M3_Pad_Via" (at 60.96 172.72 0)
+      (effects (font (size 1.27 1.27)) hide)
+    )
+    (property "Datasheet" "~" (at 60.96 172.72 0)
+      (effects (font (size 1.27 1.27)) hide)
+    )
+    (property "Description" "Mounting Hole without connection" (at 60.96 172.72 0)
+      (effects (font (size 1.27 1.27)) hide)
+    )
+    (instances
+      (project "Wideband_v3"
+        (path "/08893845-3ad0-4661-81a4-b965d2c3e6dc/3737bf71-68b2-46c2-b6f0-6262322b912b"
+          (reference "H3") (unit 1)
+        )
+      )
+    )
+  )
   (symbol (lib_id "Connector:TestPoint") (at 182.88 123.19 0) (unit 1)
     (exclude_from_sim no) (in_bom yes) (on_board yes) (dnp no) (fields_autoplaced)
@@
       (effects (font (size 1.27 1.27)) (justify left) hide)
     )
-    (property "Footprint" "Button_Switch_THT:SW_SPST_Omron_B3F-315x_Angled" (at 35.56 64.77 0)
-      (effects (font (size 1.27 1.27)) hide)
-    )
+    (property "Footprint" "Button_Switch_SMD:SW_Push_1P1T_XKB_TS-1187A" (at 35.56 64.77 0)
+      (effects (font (size 1.27 1.27)) hide)
+    )

Commit message: init 7seg pcb
Parts:
- removed TP1: SWCLK, TestPoint:TestPoint_Pad_1.0x1.0mm, symbol Connector:TestPoint
- removed TP2: SWD, TestPoint:TestPoint_Pad_1.0x1.0mm, symbol Connector:TestPoint
- added D1: B120-E3, Diode_SMD:D_SMA, symbol Diode:B120-E3
- added R5: 10k, Resistor_SMD:R_0603_1608Metric, symbol Device:R
Connections:
- net GPIO10 is gone; now on net GPIO16: J1.7 (Pin_7)
- net +3V3: now also R5.1; no longer U1.26 (RUN)
- net +5V: now also J1.11 (Pin_11), D1.1 (K)
- net NRST: now also U1.26 (RUN), R5.2
- net SYS_SWCLK: now also U1.24 (SWCLK)
- net SYS_SWDIO: now also U1.25 (SWD)
- net VBUS: now also D1.2 (A); no longer J1.11 (Pin_11)
Other:
- moved on the sheet: J1

Commit message: Cosas
Parts:
- renumbered C21 to C20, C24 to C21, C25 to C22, C28 to C23, C31 to C24, R5 to R19
Connections:
- net +3V3: no longer J1.10 (Pin_10)
- net GPIO11: no longer J1.6 (Pin_6)
- net GPIO12: no longer J1.5 (Pin_5)
- net GPIO14: now also J1.9 (Pin_9); no longer J1.4 (Pin_4)
- net GPIO19: now also J1.4 (Pin_4)
- net GPIO20: now also J1.3 (Pin_3)
- net GPIO21: now also J1.2 (Pin_2); no longer J1.3 (Pin_3)
- net GPIO26: no longer J1.2 (Pin_2)
- net GPIO7: no longer J1.9 (Pin_9)
- net GPIO8: no longer J1.8 (Pin_8)
- net FORCE_BOOTLOADER: now reaches SW1.2
- net FORCE_BOOTLOADER: now also JP4.2 (B), R6.2; no longer U1.18 (GPIO15)
- net GPIO17: now reaches U1.28 (GPIO17)
- net GPIO17: now also J1.6 (Pin_6)
- net BTN_YES: now reaches SW3.2
- net BTN_YES: now also U1.5 (GPIO3); no longer U1.29 (GPIO18)
- new net +12VA: J1.10 (Pin_10)
- new net GPIO15: J1.8 (Pin_8), U1.18 (GPIO15)
- new net GPIO18: J1.5 (Pin_5), U1.29 (GPIO18)
- no-connect marks 5 -> 7
Other:
- moved on the sheet: SW1
