File: pcb/wideband_v3/Wideband_v3/power.kicad_sch (KiCad schematic)
At the start: 10 parts, among them Q6 MCQ9435-TP, U11 LM78M05_TO252

Commit message: update DAC for v3
Parts:
- JP5: now left out of the parts list
Changed lines of the file:
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@@
 		(unit 1)
 		(exclude_from_sim no)
-		(in_bom yes)
+		(in_bom no)
 		(on_board yes)
 		(dnp no)

Commit message: update LCSC/Stock codes, update pcb to new footprints
Parts:
- C28, C29: STOCK (none) -> CAP-000202-00
- C30: STOCK (none) -> CAP-000397-00
- D10: value D_TVS -> SMCJ24CA; STOCK (none) -> DIO-000284-00
- D11: LCSC (none) -> C550392; STOCK (none) -> DIO-000398-00
- D2: LCSC (none) -> C84343; STOCK (none) -> DIO-000134-00
- JP5: LCSC (none) -> -; STOCK (none) -> -; now not fitted
- Q6: LCSC (none) -> C586650; STOCK (none) -> TRA-000400-00
- R20: LCSC C25804 -> C115324; STOCK (none) -> RES-000118-00
- U11: STOCK (none) -> PWR-000358-00
Changed lines of the file:
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@@
 	(version 20231120)
 	(generator "eeschema")
-	(generator_version "7.99")
+	(generator_version "8.0")
 	(paper "A4")
 	(title_block
@@
 			)
 		)
+		(property "STOCK" "DIO-000134-00"
+			(at 220.98 60.96 0)
+			(effects
+				(font
+					(size 1.27 1.27)
+				)
+				(hide yes)
+			)
+		)
+		(property "LCSC" "C84343"
+			(at 220.98 60.96 0)
+			(effects
+				(font
+					(size 1.27 1.27)
+				)
+				(hide yes)
+			)
+		)
 		(pin "1"
 		)
@@
 			)
 		)
+		(property "STOCK" "DIO-000398-00"
+			(at 203.2 99.06 0)
+			(effects
+				(font
+					(size 1.27 1.27)
+				)
+				(hide yes)
+			)
+		)
+		(property "LCSC" "C550392"
+			(at 203.2 99.06 0)
+			(effects
+				(font
+					(size 1.27 1.27)
+				)
+				(hide yes)
+			)
+		)
 		(pin "1"
 		)
@@
 			)
 		)
+		(property "STOCK" "PWR-000358-00"
+			(at 193.04 60.96 0)
+			(effects
+				(font
+					(size 1.27 1.27)
+				)
+				(hide yes)
+			)
+		)
 		(pin "1"
 		)
@@
 			)
 		)
+		(property "STOCK" "CAP-000202-00"
+			(at 179.705 67.31 0)
+			(effects
+				(font
+					(size 1.27 1.27)
+				)
+				(hide yes)
+			)
+		)
 		(pin "1"
 		)
@@
 		(in_bom no)
 		(on_board yes)
-		(dnp no)
+		(dnp yes)
 		(property "Reference" "JP5"
 			(at 173.99 119.888 0)
@@
 		)
 		(property "Description" ""
+			(at 173.99 121.92 0)
+			(effects
+				(font
+					(size 1.27 1.27)
+				)
+				(hide yes)
+			)
+		)
+		(property "STOCK" "-"
+			(at 173.99 121.92 0)
+			(effects
+				(font
+					(size 1.27 1.27)
+				)
+				(hide yes)
+			)
+		)
+		(property "LCSC" "-"
 			(at 173.99 121.92 0)
 			(effects
@@
 			)
 		)
+		(property "STOCK" "CAP-000397-00"
+			(at 217.805 67.31 0)
+			(effects
+				(font
+					(size 1.27 1.27)
+				)
+				(hide yes)
+			)
+		)
 		(pin "1"
 		)
@@
 			)
 		)
+		(property "STOCK" "TRA-000400-00"
+			(at 195.58 95.25 0)
+			(effects
+				(font
+					(size 1.27 1.27)
+				)
+				(hide yes)
+			)
+		)
+		(property "LCSC" "C586650"
+			(at 195.58 95.25 0)
+			(effects
+				(font
+					(size 1.27 1.27)
+				)
+				(hide yes)
+			)
+		)
 		(pin "1"
 		)
@@
 			)
 		)
-		(property "Value" "D_TVS"
+		(property "Value" "SMCJ24CA"
 			(at 187.4266 98.933 90)
 			(effects
@@
 		)
 		(property "LCSC" "C151279"
+			(at 185.42 97.79 0)
+			(effects
+				(font
+					(size 1.27 1.27)
+				)
+				(hide yes)
+			)
+		)
+		(property "STOCK" "DIO-000284-00"
 			(at 185.42 97.79 0)
 			(effects
@@
 			)
 		)
+		(property "STOCK" "CAP-000202-00"
+			(at 206.375 67.31 0)
+			(effects
+				(font
+					(size 1.27 1.27)
+				)
+				(hide yes)
+			)
+		)
 		(pin "1"
 		)
@@
 			)
 		)
-		(property "LCSC" "C25804"
+		(property "LCSC" "C115324"
 			(at 198.12 107.95 0)
 			(effects
 				(font
+					(size 1.27 1.27)
+				)
+				(hide yes)
+			)
+		)
+		(property "STOCK" "RES-000118-00"
+			(at 195.58 107.95 0)
+			(effects
+				(font
