File: pcb/wideband_v3/displays/7_Segment_LED_v1/7_Segment_LED_v1.kicad_pcb (KiCad board)
At the start: 2 copper layers, 80 x 50 mm, 24 parts, among them J1 Conn_01x14, Q1 SS8050, Q2 SS8050, Q3 SS8050, Q4 SS8050, U5 4511

Commit message: reorganize rev3 diagram, add display code to carrier fw
Parts:
- moved G*** 26.1 mm to (185.9, 97.9)
Changed lines of the file:
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@@
 (kicad_pcb
-	(version 20231014)
+	(version 20240108)
 	(generator "pcbnew")
-	(generator_version "7.99")
+	(generator_version "8.0")
 	(general
 		(thickness 1.6)
@@
 				(type "Bottom Silk Screen")
 			)
+			(layer "F.SilkS"
+				(type "Top Silk Screen")
+			)
+			(layer "F.Paste"
+				(type "Top Solder Paste")
+			)
+			(layer "F.Mask"
+				(type "Top Solder Mask")
+				(thickness 0.01)
+			)
+			(layer "F.Cu"
+				(type "copper")
+				(thickness 0.035)
+			)
+			(layer "dielectric 2"
+				(type "core")
+				(thickness 1.51)
+				(material "FR4")
+				(epsilon_r 4.5)
+				(loss_tangent 0.02)
+			)
+			(layer "B.Cu"
+				(type "copper")
+				(thickness 0.035)
+			)
+			(layer "B.Mask"
+				(type "Bottom Solder Mask")
+				(thickness 0.01)
+			)
+			(layer "B.Paste"
+				(type "Bottom Solder Paste")
+			)
+			(layer "B.SilkS"
+				(type "Bottom Silk Screen")
+			)
+			(layer "F.SilkS"
+				(type "Top Silk Screen")
+			)
+			(layer "F.Paste"
+				(type "Top Solder Paste")
+			)
+			(layer "F.Mask"
+				(type "Top Solder Mask")
+				(thickness 0.01)
+			)
+			(layer "F.Cu"
+				(type "copper")
+				(thickness 0.035)
+			)
+			(layer "dielectric 3"
+				(type "core")
+				(thickness 1.51)
+				(material "FR4")
+				(epsilon_r 4.5)
+				(loss_tangent 0.02)
+			)
+			(layer "B.Cu"
+				(type "copper")
+				(thickness 0.035)
+			)
+			(layer "B.Mask"
+				(type "Bottom Solder Mask")
+				(thickness 0.01)
+			)
+			(layer "B.Paste"
+				(type "Bottom Solder Paste")
+			)
+			(layer "B.SilkS"
+				(type "Bottom Silk Screen")
+			)
 			(copper_finish "None")
 			(dielectric_constraints no)
@@
 		)
 	)
-	(footprint "MountingHole:MountingHole_3.2mm_M3_Pad_Via" locked
+	(footprint "MountingHole:MountingHole_3.2mm_M3_Pad_Via"
+		(locked yes)
 		(layer "F.Cu")
 		(at 130.664 80.395)
@@
 	)
 	(footprint "Connector_PinHeader_2.00mm:PinHeader_2x12_P2.00mm_Vertical"
-		locked
-		(layer "F.Cu"
-		)
+		(locked yes)
+		(layer "F.Cu")
 		(at 163.679 99.77)
 		(descr "Through hole straight pin header, 2x12, 2.00mm pitch, double rows")
@@
 		)
 	)
-	(footprint "MountingHole:MountingHole_3.2mm_M3_Pad_Via" locked
+	(footprint "MountingHole:MountingHole_3.2mm_M3_Pad_Via"
+		(locked yes)
 		(layer "F.Cu")
 		(at 130.664 120.395)
@@
 		)
 	)
-	(footprint "MountingHole:MountingHole_3.2mm_M3_Pad_Via" locked
+	(footprint "MountingHole:MountingHole_3.2mm_M3_Pad_Via"
+		(locked yes)
 		(layer "F.Cu")
 		(at 200.664 120.395)
@@
 		)
 	)
-	(footprint "MountingHole:MountingHole_3.2mm_M3_Pad_Via" locked
+	(footprint "MountingHole:MountingHole_3.2mm_M3_Pad_Via"
+		(locked yes)
 		(layer "F.Cu")
 		(at 200.664 80.395)
@@
 	)
 	(footprint "Connector_PinHeader_2.54mm:PinHeader_2x07_P2.54mm_Vertical"
-		locked
-		(layer "F.Cu"
-		)
+		(locked yes)
+		(layer "F.Cu")
 		(at 129.389 92.77)
 		(descr "Through hole straight pin header, 2x07, 2.54mm pitch, double rows")
@@
 	(footprint "LOGO"
 		(layer "B.Cu")
-		(at 160.0048 94.5974 180)
+		(at 185.874 97.885 180)
 		(property "Reference" "G***"
 			(at 0 0 180)
@@
 	)
 	(gr_text "Diseñado en Argentina"
-		(at 165.5674 99.9822 0)
+		(at 191.404 103.655 0)
 		(layer "B.SilkS")
 		(effects
@@
 		)
 		(height 4)
-		(gr_text "50,0000 mm"
+		(gr_text "50.0000 mm"
 			(at 120.514 100.395 90)
 			(layer "Dwgs.User")
@@
 		)
 		(height -3)
-		(gr_text "80,0000 mm"
+		(gr_text "80.0000 mm"
 			(at 165.664 71.245 0)
 			(layer "Dwgs.User")
